File: hardware/papersynth.kicad_pcb (KiCad board)
At the start: 2 copper layers, 200 x 48.5 mm, 106 parts, among them J1 USB_OTG, J2 JACK_2P, J3 Micro_SD_Card_Det, J4 JACK_TRS_5PINS, J5 JACK_2P, Q1 Q_NPN_BEC, Q2 Q_NPN_BEC, SW1 SW_Push, SW2 SW_Push, U1 CP2102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

Commit message: Version sent out for manufacturing on 2017-12-20
Parts:
- BT1: value Battery_Cell -> BAT
- J4: footprint Connectors:PJ31060-I_3.5mm_Jack -> papersynth:35RASMT4BHNTRX
- moved C27 6.24 mm to (138.1, 78.7)
- moved U13 3.53 mm to (124.9, 84.1)
- moved J4 3.41 mm to (118.3, 77.7), turned to 270 degrees
- moved C33 3.28 mm to (125.6, 88.4)
- moved C34 3.28 mm to (123.8, 88.4)
- moved C22 3.26 mm to (145.4, 81.0)
- moved C28 3.26 mm to (145.4, 82.5)
- moved C21 3.22 mm to (136.6, 78.7)
- moved U8 2.99 mm to (139.7, 83.8)
- moved C19 2.90 mm to (142.6, 78.7)
- moved C18 2.56 mm to (133.2, 82.6)
- moved C29 2.56 mm to (133.2, 84.1)
- moved C30 2.56 mm to (133.2, 85.6)
- moved C17 2.48 mm to (133.2, 81.1)
- moved C32 2.42 mm to (122.3, 82.7), turned to 270 degrees
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Connections:
- J2 pad 1: Net-(J2-Pad1) -> GND
- J2 pad 3: GND -> Net-(J2-Pad3)
- J5 pad 1: Net-(J5-Pad1) -> GND
- J5 pad 3: GND -> Net-(J5-Pad3)
- R23 pad 1: Net-(J2-Pad1) -> Net-(J2-Pad2)
- R25 pad 1: Net-(J5-Pad1) -> Net-(J5-Pad2)
Routing:
- net Net-(J2-Pad2): track 0.00 -> 21.2 mm, vias 0 -> 1
- net Net-(J5-Pad2): track 0.00 -> 14.4 mm, vias 0 -> 1
- net Net-(C36-Pad2): track 9.90 -> 22.3 mm
- net Net-(J4-Pad4): track 13.8 -> 24.4 mm, vias 1 -> 3
- net Net-(C35-Pad2): track 5.85 -> 14.2 mm
- net Net-(C36-Pad1): track 32.4 -> 38.9 mm
- net Net-(C32-Pad1): track 8.61 -> 14.2 mm
- net Net-(J2-Pad1): track 3.42 -> 0.00 mm, vias 1 -> 0
- net /ESP32_MODULE/SYNC_IN: track 99.9 -> 103.2 mm
- net Net-(J5-Pad1): track 2.95 -> 0.00 mm, vias 1 -> 0
- net VUNREG: track 139.5 -> 137.3 mm
- net Net-(J2-Pad3): track 0.00 -> 2.09 mm, vias 0 -> 1
- net GND: track 347.0 -> 345.0 mm, vias 42 -> 47
- net Net-(U4-Pad8): track 34.6 -> 32.7 mm
- net +3V3: track 396.6 -> 398.5 mm, vias 20 -> 22
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